File: Filestore_E01.kicad_sch (KiCad schematic)
At the start: 148 parts, among them J1 Eco_Out, J10 Conn_02x01, J15 Conn_02x01, J16 Conn_01x03, J16_1 Conn_01x01_Pin, J16_2 Conn_01x01_Pin, J16_3 Conn_01x01_Pin, J2 Conn_02x01, J2 DIN-5, J3 1 us, J3 Conn_01x03, J3 Conn_02x01, J4 2us, J5 Conn_02x01, J6 Conn_02x01, J7 Conn_02x01, J7 Econet module, J8 Conn_02x01, Q1 BC212, Q2 BC212, Q3 BC160, Q4 BC107, Q5 Q_Photo_NPN_CE, SW3 Conn_01x02, U1 74LS139, U10 74HC157, U11 74HC30, U12 4464, U13 4464, U14 74LS139, U15 74LS245, U16 74HC74, U17 74HC74, U18 74LS139, U19 74HC273, U2 MC146818, U20 WD2793, U21 6522, U23 74LS244, U24 74LS14, U27 74LS125, U28 74LS163, U29 7416, U3 65C102, U30 7438, U31 7438, U32 74HC02, U33 74LS32, U34 74HC00, U35 74LS04, U37 74HC125, U4 27256, U5 27256, U6 74LS57, U7 74HC73, U8 74HC123, U9 74HC157, X1 32768 Hz, X2 8 MHz

Commit message: Specify bit of misc. register
Other:
- note added: "Miscellaneous functions latch bit 0 Floppy 1 (left) select bit 1 Floppy 2 (right) select bit 2 Floppy side (0|1) select bit 3 Access to NVRAM possible if set bit 4 FDC Disc Density (active low) bit 5 FDC MasterReset (active low) bit 6 FDC Test (active low) bit 7 Mode (red) LED"
Changed lines of the file:
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@@
+		)
+	)
+	(text "Miscellaneous functions latch\nbit 0  Floppy 1 (left) select\nbit 1  Floppy 2 (right) select\nbit 2  Floppy side (0|1) select\nbit 3  Access to NVRAM possible if set\nbit 4  FDC Disc Density (active low)\nbit 5  FDC MasterReset (active low)\nbit 6  FDC Test (active low)\nbit 7  Mode (red) LED"
+		(exclude_from_sim yes)
+		(at 446.024 173.99 0)
+		(effects
+			(font
+				(size 1.27 1.27)
+			)
+			(justify left)
 		)
 	)

Commit message: Electrical Rule Checker found some errors . Also missing connections to some chips. And wrong IC number
Parts:
- renumbered U11 to U33
Connections:
- net GNDD: no longer U20.1 (ENP), U20.29 (TG43)
- net VDD: now also U7.2 (~{R})
- new net: U20.1 (ENP), U20.29 (TG43)
Other:
- note added: "U29 = 7416"
Changed lines of the file:
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@@
 	)
 	(junction
-		(at 586.74 99.06)
-		(diameter 0)
-		(color 0 0 0 0)
-	)
-	(junction
 		(at 660.4 109.22)
 		(diameter 0)
@@
 	(wire
 		(pts
+			(xy 586.74 96.52) (xy 586.74 99.06)
+		)
+		(stroke
+			(width 0)
+			(type default)
+		)
+	)
+	(wire
+		(pts
 			(xy 144.78 200.66) (xy 148.59 200.66)
 		)
@@
 		)
 	)
+	(wire
+		(pts
+			(xy 134.62 218.44) (xy 134.62 222.25)
+		)
+		(stroke
+			(width 0)
+			(type default)
+		)
+	)
 	(bus
 		(pts
@@
 	(wire
 		(pts
-			(xy 586.74 99.06) (xy 586.74 100.33)
-		)
-		(stroke
-			(width 0)
-			(type default)
-		)
-	)
-	(wire
-		(pts
 			(xy 548.64 441.96) (xy 548.64 447.04)
 		)
@@
 	(wire
 		(pts
-			(xy 586.74 96.52) (xy 586.74 99.06)
-		)
-		(stroke
-			(width 0)
-			(type default)
-		)
-	)
-	(wire
-		(pts
 			(xy 753.11 210.82) (xy 774.7 210.82)
 		)
@@
 	(wire
 		(pts
+			(xy 223.52 204.47) (xy 223.52 207.01)
+		)
+		(stroke
+			(width 0)
+			(type default)
+		)
+	)
+	(wire
+		(pts
 			(xy 725.17 334.01) (xy 736.6 334.01)
 		)
@@
 	(wire
 		(pts
-			(xy 134.62 218.44) (xy 134.62 220.98)
-		)
-		(stroke
-			(width 0)
-			(type default)
-		)
-	)
-	(wire
-		(pts
 			(xy 758.19 66.04) (xy 758.19 68.58)
 		)
@@
 		)
 	)
+	(text "U29 = 7416\n"
+		(exclude_from_sim no)
+		(at 704.342 91.948 0)
+		(effects
+			(font
+				(size 1.27 1.27)
+			)
+		)
+	)
 	(text "MOS"
 		(exclude_from_sim no)
@@
 		(dnp no)
 		(fields_autoplaced yes)
-		(property "Reference" "U11"
+		(property "Reference" "U33"
 			(at 548.64 178.054 0)
 			(effects
@@
 			(project ""
 				(path "/8b1de929-f561-4d06-8ee9-44ad55095b8f"
-					(reference "U11")
+					(reference "U33")
 					(unit 4)
 				)
@@
 	(symbol
 		(lib_id "power:GNDD")
-		(at 134.62 220.98 0)
+		(at 134.62 222.25 0)
 		(unit 1)
 		(exclude_from_sim no)
@@
 		(fields_autoplaced yes)
 		(property "Reference" "#PWR089"
-			(at 134.62 227.33 0)
+			(at 134.62 228.6 0)
 			(effects
 				(font
@@
 		)
 		(property "Value" "GNDD"
-			(at 134.62 224.79 0)
+			(at 134.62 226.06 0)
 			(effects
 				(font
@@
 		)
 		(property "Footprint" ""
-			(at 134.62 220.98 0)
+			(at 134.62 222.25 0)
 			(effects
 				(font
@@
 		)
 		(property "Datasheet" ""
-			(at 134.62 220.98 0)
+			(at 134.62 222.25 0)
 			(effects
 				(font
@@
 		)
 		(property "Description" "Power symbol creates a global label with name \"GNDD\" , digital ground"
-			(at 134.62 220.98 0)
+			(at 134.62 222.25 0)
 			(effects
 				(font
@@
 	)
 	(symbol
+		(lib_id "power:VDD")
+		(at 223.52 204.47 0)
+		(unit 1)
+		(exclude_from_sim no)
+		(in_bom yes)
+		(on_board yes)
+		(dnp no)
+		(property "Reference" "#PWR0103"
+			(at 223.52 208.28 0)
+			(effects
+				(font
+					(size 1.27 1.27)
+				)
+				(hide yes)
+			)
+		)
+		(property "Value" "VDD"
+			(at 223.52 199.39 0)
+			(effects
+				(font
+					(size 1.27 1.27)
+				)
+			)
+		)
+		(property "Footprint" ""
+			(at 223.52 204.47 0)
+			(effects
+				(font
+					(size 1.27 1.27)
+				)
+				(hide yes)
+			)
+		)
+		(property "Datasheet" ""
+			(at 223.52 204.47 0)
+			(effects
+				(font
+					(size 1.27 1.27)
+				)
+				(hide yes)
+			)
+		)
+		(property "Description" "Power symbol creates a global label with name \"VDD\""
+			(at 223.52 204.47 0)
+			(effects
+				(font
+					(size 1.27 1.27)
+				)
+				(hide yes)
+			)
+		)
+		(pin "1"
+		)
+		(instances
+			(project "Filestore_E01"
+				(path "/8b1de929-f561-4d06-8ee9-44ad55095b8f"
+					(reference "#PWR0103")
+					(unit 1)
+				)
+			)
+		)
+	)
+	(symbol
 		(lib_id "power:GNDD")
 		(at 758.19 102.87 0)
@@
 					(unit 1)
 				)
-			)
-		)
-	)
-	(symbol
-		(lib_id "power:GNDD")
-		(at 586.74 100.33 0)
-		(unit 1)
-		(exclude_from_sim no)
-		(in_bom yes)
-		(on_board yes)
-		(dnp no)
-		(fields_autoplaced yes)
-		(property "Reference" "#PWR026"
-			(at 586.74 106.68 0)
-			(effects
-				(font
-					(size 1.27 1.27)
-				)
-				(hide yes)
-			)
-		)
-		(property "Value" "GNDD"
-			(at 586.74 104.14 0)
-			(effects
-				(font
-					(size 1.27 1.27)
-				)
-				(hide yes)
-			)
-		)
-		(property "Footprint" ""
-			(at 586.74 100.33 0)
-			(effects
-				(font
-					(size 1.27 1.27)
-				)
-				(hide yes)
-			)
-		)
-		(property "Datasheet" ""
-			(at 586.74 100.33 0)
-			(effects
-				(font
-					(size 1.27 1.27)
-				)
-				(hide yes)
-			)
-		)
-		(property "Description" "Power symbol creates a global label with name \"GNDD\" , digital ground"
-			(at 586.74 100.33 0)
-			(effects
-				(font
-					(size 1.27 1.27)
-				)
-				(hide yes)
-			)
-		)
-		(pin "1"
-		)
-		(instances
-			(project "Filestore_E01"
-				(path "/8b1de929-f561-4d06-8ee9-44ad55095b8f"
-					(reference "#PWR026")
-					(unit 1)
-				)
